Commit message: Modify torque feedback coefficient

File: legged_examples/legged_hunter/legged_hunter_description/urdf/hunter.urdf (robot description, URDF)
Before this commit: robot pai_12dof_v2_0312, 18 links, 17 joints
Joints:
- joint leg_l5_joint: limit lower=-0.8 upper=1.2 effort=21 velocity=21 -> lower=-1.57 upper=1.57 effort=21 velocity=21
- joint leg_r5_joint: limit lower=-1.2 upper=0.95 effort=21 velocity=21 -> lower=-1.57 upper=1.57 effort=21 velocity=21

Commit message: temp

File: legged_examples/legged_hunter/legged_hunter_description/urdf/hunter.urdf (robot description, URDF)
Before this commit: robot pai_12dof_v2_0312, 18 links, 17 joints
Links:
- link base_link: mass 1.4140796 -> 2.0

Commit message: 缩小WBC的扭矩约束

File: legged_examples/legged_hunter/legged_hunter_description/urdf/hunter.urdf (robot description, URDF)
Before this commit: robot pai_12dof_v2_0312, 18 links, 17 joints
Joints:
- joint leg_l1_joint: limit lower=-0.5 upper=1.0 effort=21 velocity=21 -> lower=-3.14 upper=3.14 effort=21 velocity=21
- joint leg_l2_joint: limit lower=-0.9 upper=2 effort=21 velocity=21 -> lower=-3.14 upper=3.14 effort=21 velocity=21
- joint leg_l3_joint: limit lower=-0.8 upper=1.8 effort=21 velocity=21 -> lower=-3.14 upper=3.14 effort=21 velocity=21
- joint leg_l4_joint: limit lower=-0.15 upper=2.0 effort=21 velocity=21 -> lower=-3.14 upper=3.14 effort=21 velocity=21
- joint leg_l5_joint: limit lower=-1.57 upper=1.57 effort=21 velocity=21 -> lower=-3.14 upper=3.14 effort=21 velocity=21
- joint leg_r1_joint: limit lower=-1.0 upper=0.5 effort=21 velocity=21 -> lower=-3.14 upper=3.14 effort=21 velocity=21
- joint leg_r2_joint: limit lower=-2 upper=0.9 effort=21 velocity=21 -> lower=-3.14 upper=3.14 effort=21 velocity=21
- joint leg_r3_joint: limit lower=-1.8 upper=0.8 effort=21 velocity=21 -> lower=-3.14 upper=3.14 effort=21 velocity=21
- joint leg_r4_joint: limit lower=-0.15 upper=2.0 effort=21 velocity=21 -> lower=-3.14 upper=3.14 effort=21 velocity=21
- joint leg_r5_joint: limit lower=-1.57 upper=1.57 effort=21 velocity=21 -> lower=-3.14 upper=3.14 effort=21 velocity=21

Commit message: urdf limit pos

File: legged_examples/legged_hunter/legged_hunter_description/urdf/hunter.urdf (robot description, URDF)
Before this commit: robot pai_12dof_v2_0312, 18 links, 17 joints
Joints:
- joint leg_l1_joint: limit lower=-3.14 upper=3.14 effort=21 velocity=21 -> lower=-0.8 upper=1.8 effort=21 velocity=21
- joint leg_l2_joint: limit lower=-3.14 upper=3.14 effort=21 velocity=21 -> lower=-0.9 upper=2 effort=21 velocity=21
- joint leg_l3_joint: limit lower=-3.14 upper=3.14 effort=21 velocity=21 -> lower=-0.8 upper=1.8 effort=21 velocity=21
- joint leg_l4_joint: limit lower=-3.14 upper=3.14 effort=21 velocity=21 -> lower=-0.15 upper=2.0 effort=21 velocity=21
- joint leg_l5_joint: limit lower=-3.14 upper=3.14 effort=21 velocity=21 -> lower=-0.8 upper=1.2 effort=21 velocity=21
- joint leg_r1_joint: limit lower=-3.14 upper=3.14 effort=21 velocity=21 -> lower=-1.0 upper=0.5 effort=21 velocity=21
- joint leg_r2_joint: limit lower=-3.14 upper=3.14 effort=21 velocity=21 -> lower=-2 upper=0.9 effort=21 velocity=21
- joint leg_r3_joint: limit lower=-3.14 upper=3.14 effort=21 velocity=21 -> lower=-1.8 upper=0.8 effort=21 velocity=21
- joint leg_r4_joint: limit lower=-3.14 upper=3.14 effort=21 velocity=21 -> lower=-0.15 upper=2.0 effort=21 velocity=21
- joint leg_r5_joint: limit lower=-3.14 upper=3.14 effort=21 velocity=21 -> lower=-1.2 upper=0.95 effort=21 velocity=21

Commit message: 真机调试

File: legged_examples/legged_hunter/legged_hunter_description/urdf/hunter.urdf (robot description, URDF)
Before this commit: robot pai_12dof_v2_0312, 18 links, 17 joints
Joints:
- joint leg_l3_joint: axis 0 -1 0 -> 0 1 0
- joint leg_l5_joint: axis 0 -1 0 -> 0 1 0; limit lower=-0.8 upper=1.2 effort=21 velocity=21 -> lower=-1.57 upper=1.57 effort=21 velocity=21
- joint leg_r5_joint: limit lower=-1.2 upper=0.95 effort=21 velocity=21 -> lower=-1.57 upper=1.57 effort=21 velocity=21

File: legged_examples/legged_hunter/legged_hunter_description/urdf/hunter_sim.urdf (robot description, URDF)
Before this commit: robot pai_12dof_v2_0312, 18 links, 17 joints
Joints:
- joint leg_l3_joint: axis 0 -1 0 -> 0 1 0
- joint leg_l5_joint: axis 0 -1 0 -> 0 1 0

Commit message: 更换新小派urdf,手动调节urdf的关节坐标偏置

File: legged_examples/legged_hunter/legged_hunter_description/urdf/hunter.urdf (robot description, URDF)
Before this commit: robot pai_12dof_v2_0312, 18 links, 17 joints
Links:
- link base_link: mass 1.4140796 -> 1.917
- link l_ankle_roll_link: mass 0.1728932 -> 0.198; geometry collision box size=0.125 0.07 0.02; visual mesh filename=package://legged_hunter_description/meshes/l_foot_link.STL
- link leg_l1_link: mass 0.74952 -> 0.444991449767726; geometry collision box size=0.0001 0.0001 0.0001; visual mesh filename=package://legged_hunter_description/meshes/l_kuan_link.STL
- link leg_l2_link: mass 0.3887654 -> 0.81414; geometry collision box size=0.0001 0.0001 0.0001; visual mesh filename=package://legged_hunter_description/meshes/l_kuan2_link.STL
- link leg_l3_link: mass 0.1443603 -> 0.224
- link leg_l4_link: mass 0.768122 -> 0.538
- link leg_l5_link: geometry collision box size=0.00 0.00 0.00; visual mesh filename=package://legged_hunter_description/meshes/l_ankle_link.STL
- link leg_r1_link: mass 0.7495221 -> 0.44499; geometry collision box size=0.0001 0.0001 0.0001; visual mesh filename=package://legged_hunter_description/meshes/r_kuan_link.STL
- link leg_r2_link: mass 0.3887654 -> 0.81414; geometry collision box size=0.0001 0.0001 0.0001; visual mesh filename=package://legged_hunter_description/meshes/r_kuan2_link.STL
- link leg_r3_link: mass 0.1443603 -> 0.224
- link leg_r4_link: mass 0.768122 -> 0.444942664885023
- link leg_r5_link: mass 0.0088647 -> 0.00886465357060087; geometry collision box size=0.0 0.0 0.0; visual mesh filename=package://legged_hunter_description/meshes/r_ankle_link.STL
- link r_ankle_roll_link: mass 0.1728932 -> 0.198; geometry collision box size=0.125 0.07 0.02; visual mesh filename=package://legged_hunter_description/meshes/r_foot_link.STL
Joints:
- joint leg_l1_joint: axis 1 0 0 -> 0 0 1; limit lower=-0.5 upper=1.0 effort=21 velocity=21 -> lower=-3.14 upper=3.14 effort=21 velocity=21; origin xyz=-0.04 0 -0.05 rpy=0 0 0 -> xyz=-0.003125 0.075 -0.009 rpy=0 0 0; parent leg_l2_link -> base_link
- joint leg_l2_joint: axis 0 0 1 -> 1 0 0; limit lower=-0.9 upper=2 effort=21 velocity=21 -> lower=-3.14 upper=3.14 effort=21 velocity=21; origin xyz=0 0.075 0 rpy=0 0 0 -> xyz=-0.035 0 -0.056 rpy=0 0 0; parent base_link -> leg_l1_link
- joint leg_l3_joint: limit lower=-0.8 upper=1.8 effort=21 velocity=21 -> lower=-3.14 upper=3.14 effort=21 velocity=21; origin xyz=0.04 0 0 rpy=0 0 0 -> xyz=0.035 0 0 rpy=0 0 0; parent leg_l1_link -> leg_l2_link
- joint leg_l4_joint: limit lower=-0.15 upper=2.0 effort=21 velocity=21 -> lower=-3.14 upper=3.14 effort=21 velocity=21; origin xyz=0.014 0 -0.14935 rpy=0 0 0 -> xyz=0.0075 0 -0.14981 rpy=0 0 0
- joint leg_l5_fixed_1: origin xyz=0.1 0 -0.0100 rpy=0 0 0 -> xyz=0.07 0 -0.030 rpy=0 0 0
- joint leg_l5_fixed_2: origin xyz=-0.04 0 -0.0100 rpy=0 0 0 -> xyz=-0.055 0 -0.0300 rpy=0 0 0
- joint leg_l5_joint: limit lower=-1.57 upper=1.57 effort=21 velocity=21 -> lower=-3.14 upper=3.14 effort=21 velocity=21; origin xyz=0.0025 0 -0.15845 rpy=0 0 0 -> xyz=0 -0.001 -0.17495 rpy=0 0 0
- joint leg_r1_joint: axis 1 0 0 -> 0 0 1; limit lower=-1.0 upper=0.5 effort=21 velocity=21 -> lower=-3.14 upper=3.14 effort=21 velocity=21; origin xyz=-0.04 0 -0.05 rpy=0 0 0 -> xyz=-0.003125 -0.075 -0.009 rpy=0 0 0; parent leg_r2_link -> base_link
- joint leg_r2_joint: axis 0 0 1 -> 1 0 0; limit lower=-2 upper=0.9 effort=21 velocity=21 -> lower=-3.14 upper=3.14 effort=21 velocity=21; origin xyz=0 -0.075 0 rpy=0 0 0 -> xyz=-0.035 0 -0.056 rpy=0 0 0; parent base_link -> leg_r1_link
- joint leg_r3_joint: limit lower=-1.8 upper=0.8 effort=21 velocity=21 -> lower=-3.14 upper=3.14 effort=21 velocity=21; origin xyz=0.04 0 0 rpy=0 0 0 -> xyz=0.035 0 0 rpy=0 0 0; parent leg_r1_link -> leg_r2_link
- joint leg_r4_joint: limit lower=-0.15 upper=2.0 effort=21 velocity=21 -> lower=-3.14 upper=3.14 effort=21 velocity=21; origin xyz=0.014 0 -0.14935 rpy=0 0 0 -> xyz=0.0075 0.0 -0.14981 rpy=0 0 0
- joint leg_r5_fixed_1: origin xyz=0.1 0 -0.0100 rpy=0 0 0 -> xyz=0.07 0 -0.030 rpy=0 0 0
- joint leg_r5_fixed_2: origin xyz=-0.040 0 -0.0100 rpy=0 0 0 -> xyz=-0.055 0 -0.0300 rpy=0 0 0
- joint leg_r5_joint: limit lower=-1.57 upper=1.57 effort=21 velocity=21 -> lower=-3.14 upper=3.14 effort=21 velocity=21; origin xyz=0.0025 0 -0.15845 rpy=0 0 0 -> xyz=0 0.001 -0.17495 rpy=0 0 0

File: legged_examples/legged_hunter/legged_hunter_description/urdf/hunter_sim.urdf (robot description, URDF)
Before this commit: robot pai_12dof_v2_0312, 18 links, 17 joints
Links:
- link base_link: mass 1.4140796 -> 1.917
- link l_ankle_roll_link: mass 0.1728932 -> 0.198; geometry collision box size=0.125 0.07 0.02; visual mesh filename=package://legged_hunter_description/meshes/l_foot_link.STL
- link leg_l1_link: mass 0.74952 -> 0.444991449767726; geometry collision box size=0.0001 0.0001 0.0001; visual mesh filename=package://legged_hunter_description/meshes/l_kuan_link.STL
- link leg_l2_link: mass 0.3887654 -> 0.81414; geometry collision box size=0.0001 0.0001 0.0001; visual mesh filename=package://legged_hunter_description/meshes/l_kuan2_link.STL
- link leg_l3_link: mass 0.1443603 -> 0.224
- link leg_l4_link: mass 0.768122 -> 0.538
- link leg_l5_link: geometry collision box size=0.00 0.00 0.00; visual mesh filename=package://legged_hunter_description/meshes/l_ankle_link.STL
- link leg_r1_link: mass 0.7495221 -> 0.44499; geometry collision box size=0.0001 0.0001 0.0001; visual mesh filename=package://legged_hunter_description/meshes/r_kuan_link.STL
- link leg_r2_link: mass 0.3887654 -> 0.81414; geometry collision box size=0.0001 0.0001 0.0001; visual mesh filename=package://legged_hunter_description/meshes/r_kuan2_link.STL
- link leg_r3_link: mass 0.1443603 -> 0.224
- link leg_r4_link: mass 0.768122 -> 0.444942664885023
- link leg_r5_link: mass 0.0088647 -> 0.00886465357060087; geometry collision box size=0.0 0.0 0.0; visual mesh filename=package://legged_hunter_description/meshes/r_ankle_link.STL
- link r_ankle_roll_link: mass 0.1728932 -> 0.198; geometry collision box size=0.125 0.07 0.02; visual mesh filename=package://legged_hunter_description/meshes/r_foot_link.STL
Joints:
- joint leg_l1_joint: axis 1 0 0 -> 0 0 1; limit lower=-0.5 upper=1.0 effort=21 velocity=21 -> lower=-3.14 upper=3.14 effort=21 velocity=21; origin xyz=-0.04 0 -0.05 rpy=0 0 0 -> xyz=-0.003125 0.075 -0.009 rpy=0 0 0; parent leg_l2_link -> base_link
- joint leg_l2_joint: axis 0 0 1 -> 1 0 0; limit lower=-0.9 upper=2 effort=21 velocity=21 -> lower=-3.14 upper=3.14 effort=21 velocity=21; origin xyz=0 0.075 0 rpy=0 0 0 -> xyz=-0.035 0 -0.056 rpy=0 0 0; parent base_link -> leg_l1_link
- joint leg_l3_joint: limit lower=-0.8 upper=1.8 effort=21 velocity=21 -> lower=-3.14 upper=3.14 effort=21 velocity=21; origin xyz=0.04 0 0 rpy=0 0 0 -> xyz=0.035 0 0 rpy=0 0 0; parent leg_l1_link -> leg_l2_link
- joint leg_l4_joint: limit lower=-0.15 upper=2.0 effort=21 velocity=21 -> lower=-3.14 upper=3.14 effort=21 velocity=21; origin xyz=0.014 0 -0.14935 rpy=0 0 0 -> xyz=0.0075 0 -0.14981 rpy=0 0 0
- joint leg_l5_fixed_1: origin xyz=0.1 0 -0.0100 rpy=0 0 0 -> xyz=0.07 0 -0.030 rpy=0 0 0
- joint leg_l5_fixed_2: origin xyz=-0.04 0 -0.0100 rpy=0 0 0 -> xyz=-0.055 0 -0.0300 rpy=0 0 0
- joint leg_l5_joint: limit lower=-0.8 upper=1.2 effort=21 velocity=21 -> lower=-3.14 upper=3.14 effort=21 velocity=21; origin xyz=0.0025 0 -0.15845 rpy=0 0 0 -> xyz=0 -0.001 -0.17495 rpy=0 0 0
- joint leg_r1_joint: axis 1 0 0 -> 0 0 1; limit lower=-1.0 upper=0.5 effort=21 velocity=21 -> lower=-3.14 upper=3.14 effort=21 velocity=21; origin xyz=-0.04 0 -0.05 rpy=0 0 0 -> xyz=-0.003125 -0.075 -0.009 rpy=0 0 0; parent leg_r2_link -> base_link
- joint leg_r2_joint: axis 0 0 1 -> 1 0 0; limit lower=-2 upper=0.9 effort=21 velocity=21 -> lower=-3.14 upper=3.14 effort=21 velocity=21; origin xyz=0 -0.075 0 rpy=0 0 0 -> xyz=-0.035 0 -0.056 rpy=0 0 0; parent base_link -> leg_r1_link
- joint leg_r3_joint: limit lower=-1.8 upper=0.8 effort=21 velocity=21 -> lower=-3.14 upper=3.14 effort=21 velocity=21; origin xyz=0.04 0 0 rpy=0 0 0 -> xyz=0.035 0 0 rpy=0 0 0; parent leg_r1_link -> leg_r2_link
- joint leg_r4_joint: limit lower=-0.15 upper=2.0 effort=21 velocity=21 -> lower=-3.14 upper=3.14 effort=21 velocity=21; origin xyz=0.014 0 -0.14935 rpy=0 0 0 -> xyz=0.0075 0.0 -0.14981 rpy=0 0 0
- joint leg_r5_fixed_1: origin xyz=0.1 0 -0.0100 rpy=0 0 0 -> xyz=0.07 0 -0.030 rpy=0 0 0
- joint leg_r5_fixed_2: origin xyz=-0.040 0 -0.0100 rpy=0 0 0 -> xyz=-0.055 0 -0.0300 rpy=0 0 0
- joint leg_r5_joint: limit lower=-1.2 upper=0.95 effort=21 velocity=21 -> lower=-3.14 upper=3.14 effort=21 velocity=21; origin xyz=0.0025 0 -0.15845 rpy=0 0 0 -> xyz=0 0.001 -0.17495 rpy=0 0 0

File: legged_examples/legged_hunter/legged_hunter_description/urdf/mujoco/hunter.urdf (robot description, URDF)
Before this commit: robot pai_12dof_v2_0312, 15 links, 14 joints
Links:
- added link l_ankle_roll_link, mass 0.198; collision box size=0.125 0.07 0.02; visual mesh filename=package://legged_hunter_description/meshes/l_foot_link.STL
- added link leg_l_f1_link, mass 0.01; collision sphere radius=0.001; visual sphere radius=0.001
- added link r_ankle_roll_link, mass 0.198; collision box size=0.125 0.07 0.02; visual mesh filename=package://legged_hunter_description/meshes/r_foot_link.STL
- link base_link: mass 1.4140796 -> 1.917; geometry collision box size=0.2 0.2 0.12; visual mesh filename=package://legged_hunter_description/meshes/base_link.STL
- link leg_l1_link: mass 0.74952 -> 0.444991449767726; geometry collision box size=0.0001 0.0001 0.0001; visual mesh filename=package://legged_hunter_description/meshes/l_kuan_link.STL
- link leg_l2_link: mass 0.19436 -> 0.81414; geometry collision box size=0.0001 0.0001 0.0001; visual mesh filename=package://legged_hunter_description/meshes/l_kuan2_link.STL
- link leg_l3_link: mass 0.1443603 -> 0.224; geometry collision box size=0.01 0.01 0.09; visual mesh filename=package://legged_hunter_description/meshes/l_thigh_link.STL
- link leg_l4_link: mass 0.768122 -> 0.538; geometry collision box size=0.01 0.01 0.09; visual mesh filename=package://legged_hunter_description/meshes/l_calf_link.STL
- link leg_l5_link: geometry collision box size=0.00 0.00 0.00; visual mesh filename=package://legged_hunter_description/meshes/l_ankle_link.STL
- link leg_r1_link: mass 0.7495221 -> 0.44499; geometry collision box size=0.0001 0.0001 0.0001; visual mesh filename=package://legged_hunter_description/meshes/r_kuan_link.STL
- link leg_r2_link: mass 0.3887654 -> 0.81414; geometry collision box size=0.0001 0.0001 0.0001; visual mesh filename=package://legged_hunter_description/meshes/r_kuan2_link.STL
- link leg_r3_link: mass 0.1443603 -> 0.224; geometry collision box size=0.01 0.01 0.09; visual mesh filename=package://legged_hunter_description/meshes/r_thigh_link.STL
- link leg_r4_link: mass 0.768122 -> 0.444942664885023; geometry collision box size=0.01 0.01 0.09; visual mesh filename=package://legged_hunter_description/meshes/r_calf_link.STL
- link leg_r5_link: mass 0.0088647 -> 0.00886465357060087; geometry collision box size=0.0 0.0 0.0; visual mesh filename=package://legged_hunter_description/meshes/r_ankle_link.STL
Joints:
- added joint l_ankle_roll_joint: type fixed, parent leg_l5_link, child l_ankle_roll_link, origin xyz=0 0 0 rpy=0 0 0
- added joint leg_l5_fixed_1: type fixed, parent l_ankle_roll_link, child leg_l_f1_link, origin xyz=0.07 0 -0.030 rpy=0 0 0
- added joint r_ankle_roll_joint: type fixed, parent leg_r5_link, child r_ankle_roll_link, origin xyz=0 0 0 rpy=0 0 0
- joint leg_l1_joint: axis 1 0 0 -> 0 0 1; limit lower=-0.2 upper=0.5 effort=21 velocity=21 -> lower=-3.14 upper=3.14 effort=21 velocity=21; origin xyz=-0.04 0 -0.05 rpy=0 0 0 -> xyz=-0.003125 0.075 -0.009 rpy=0 0 0; parent leg_l2_link -> base_link
- joint leg_l2_joint: axis 0 0 1 -> 1 0 0; limit lower=-0.5 upper=1.5 effort=21 velocity=21 -> lower=-3.14 upper=3.14 effort=21 velocity=21; origin xyz=0 0.075 0 rpy=0 0 0 -> xyz=-0.035 0 -0.056 rpy=0 0 0; parent base_link -> leg_l1_link
- joint leg_l3_joint: axis 0 -1 0 -> 0 1 0; limit lower=-0.8 upper=1.2 effort=21 velocity=21 -> lower=-3.14 upper=3.14 effort=21 velocity=21; origin xyz=0.04 0 0 rpy=0 0 0 -> xyz=0.035 0 0 rpy=0 0 0; parent leg_l1_link -> leg_l2_link
- joint leg_l4_joint: limit lower=0 upper=1.5 effort=21 velocity=21 -> lower=-3.14 upper=3.14 effort=21 velocity=21; origin xyz=0.014 0 -0.14935 rpy=0 0 0 -> xyz=0.0075 0 -0.14981 rpy=0 0 0
- joint leg_l5_fixed_2: origin xyz=-0.030 0 -0.007 rpy=0 0 0 -> xyz=-0.055 0 -0.0300 rpy=0 0 0; parent leg_l5_link -> l_ankle_roll_link
- joint leg_l5_joint: axis 0 -1 0 -> 0 1 0; limit lower=-0.7 upper=0.4 effort=21 velocity=21 -> lower=-3.14 upper=3.14 effort=21 velocity=21; origin xyz=0.0025 0 -0.15845 rpy=0 0 0 -> xyz=0 -0.001 -0.17495 rpy=0 0 0
- joint leg_r1_joint: axis 1 0 0 -> 0 0 1; limit lower=-0.5 upper=0.2 effort=21 velocity=21 -> lower=-3.14 upper=3.14 effort=21 velocity=21; origin xyz=-0.04 0 -0.05 rpy=0 0 0 -> xyz=-0.003125 -0.075 -0.009 rpy=0 0 0; parent leg_r2_link -> base_link
- joint leg_r2_joint: axis 0 0 1 -> 1 0 0; limit lower=-1.5 upper=0.5 effort=21 velocity=21 -> lower=-3.14 upper=3.14 effort=21 velocity=21; origin xyz=0 -0.075 0 rpy=0 0 0 -> xyz=-0.035 0 -0.056 rpy=0 0 0; parent base_link -> leg_r1_link
- joint leg_r3_joint: limit lower=-1.2 upper=0.8 effort=21 velocity=21 -> lower=-3.14 upper=3.14 effort=21 velocity=21; origin xyz=0.04 0 0 rpy=0 0 0 -> xyz=0.035 0 0 rpy=0 0 0; parent leg_r1_link -> leg_r2_link
- joint leg_r4_joint: limit lower=0 upper=1.5 effort=21 velocity=21 -> lower=-3.14 upper=3.14 effort=21 velocity=21; origin xyz=0.014 0 -0.14935 rpy=0 0 0 -> xyz=0.0075 0.0 -0.14981 rpy=0 0 0
- joint leg_r5_fixed_1: origin xyz=0.06 0 -0.007 rpy=0 0 0 -> xyz=0.07 0 -0.030 rpy=0 0 0; parent leg_r5_link -> r_ankle_roll_link
- joint leg_r5_fixed_2: origin xyz=-0.030 0 -0.007 rpy=0 0 0 -> xyz=-0.055 0 -0.0300 rpy=0 0 0; parent leg_r5_link -> r_ankle_roll_link
- joint leg_r5_joint: limit lower=-0.4 upper=0.7 effort=21 velocity=21 -> lower=-3.14 upper=3.14 effort=21 velocity=21; origin xyz=0.0025 0 -0.15845 rpy=0 0 0 -> xyz=0 0.001 -0.17495 rpy=0 0 0

Commit message: 切换到新小pi上开发，保存一下旧版小派的代码

File: legged_examples/legged_hunter/legged_hunter_description/urdf/hunter.urdf (robot description, URDF)
Before this commit: robot pai_12dof_v2_0312, 18 links, 17 joints
Joints:
- joint leg_l5_fixed_1: origin xyz=0.1 0 -0.0100 rpy=0 0 0 -> xyz=0.09 0 -0.0100 rpy=0 0 0
- joint leg_r5_fixed_1: origin xyz=0.1 0 -0.0100 rpy=0 0 0 -> xyz=0.09 0 -0.0100 rpy=0 0 0

Commit message: 任务同步

File: legged_examples/legged_hunter/legged_hunter_description/urdf/hunter.urdf (robot description, URDF)
Before this commit: robot pai_12dof_v2_0312, 18 links, 17 joints
Joints:
- joint leg_l5_fixed_1: origin xyz=0.07 0 -0.030 rpy=0 0 0 -> xyz=0.07 0 -0.010 rpy=0 0 0
- joint leg_l5_fixed_2: origin xyz=-0.055 0 -0.0300 rpy=0 0 0 -> xyz=-0.055 0 -0.01 rpy=0 0 0
- joint leg_r5_fixed_1: origin xyz=0.07 0 -0.030 rpy=0 0 0 -> xyz=0.07 0 -0.010 rpy=0 0 0
- joint leg_r5_fixed_2: origin xyz=-0.055 0 -0.0300 rpy=0 0 0 -> xyz=-0.055 0 -0.01 rpy=0 0 0
